Commit message: added ur5_control and ur5 packages

File: ur5/urdf/rviz/ur5.urdf.xacro (robot description, xacro)
@@ -1,7 +1,14 @@
 <?xml version="1.0"?>
 <robot xmlns:xacro="http://www.ros.org/wiki/xacro">
+<!--
+Modified by Qianli Ma
+01/15/2015
+.dae -> .stl for collision/geometry/meshes
+-->
   <xacro:include filename="$(find ur_description)/urdf/ur5.transmission.xacro" />
   <xacro:include filename="$(find ur_description)/urdf/ur5.gazebo.xacro" />
+  <!-- materials.urdf.xacro
   <xacro:include filename="$(find ur_description)/urdf/materials.urdf.xacro" />
+   -->
 <!--
 DH for UR5:
@@ -53,5 +60,5 @@
 	<collision>
       <geometry>
-        <mesh filename="package://ur_description/meshes/ur5/collision/Base.dae" />
+        <mesh filename="package://ur_description/meshes/ur5/collision/base.stl" />
       </geometry>
       <!-- <origin rpy="0.0 0.0 0.0" xyz="0.0 0.0 -0.009159"/> -->
@@ -78,5 +85,5 @@
     <collision>
       <geometry>
-        <mesh filename="package://ur_description/meshes/ur5/collision/Shoulder.dae" />
+        <mesh filename="package://ur_description/meshes/ur5/collision/shoulder.stl" />
       </geometry>
       <!-- <origin rpy="0.0 0.0 0.0" xyz="0.0 0.0 -0.009159"/> -->
@@ -105,5 +112,5 @@
     <collision>
       <geometry>
-        <mesh filename="package://ur_description/meshes/ur5/collision/UpperArm.dae" />
+        <mesh filename="package://ur_description/meshes/ur5/collision/upper_arm.stl" />
       </geometry>
 <!--       <origin rpy="0.0 0.0 0.0" xyz="0.0 0.0 0.2125"/> -->
@@ -131,5 +138,5 @@
     <collision>
       <geometry>
-        <mesh filename="package://ur_description/meshes/ur5/collision/Forearm.dae" />
+        <mesh filename="package://ur_description/meshes/ur5/collision/forearm.stl" />
       </geometry>
 <!--       <origin rpy="0.0 0.0 0.0" xyz="0.0 0.0 0.196125"/> -->
@@ -158,5 +165,5 @@
     <collision>
       <geometry>
-        <mesh filename="package://ur_description/meshes/ur5/collision/Wrist1.dae" />
+        <mesh filename="package://ur_description/meshes/ur5/collision/wrist_1.stl" />
       </geometry>
       <origin rpy="0.0 1.570796325 0.0" xyz="0.0 0.093 0.0"/>
@@ -185,5 +192,5 @@
     <collision>
       <geometry>
-        <mesh filename="package://ur_description/meshes/ur5/collision/Wrist2.dae" />
+        <mesh filename="package://ur_description/meshes/ur5/collision/wrist_2.stl" />
       </geometry>
        <origin rpy="0.0 0.0 0.0" xyz="0.0 0.0 0.09465"/>
@@ -211,5 +218,5 @@
     <collision>
       <geometry>
-        <mesh filename="package://ur_description/meshes/ur5/collision/Wrist3.dae" />
+        <mesh filename="package://ur_description/meshes/ur5/collision/wrist_3.stl" />
       </geometry>
     </collision>
