Commit message: Transfer changes in active_echo branch to master

File: sensor_description/urdf/ur5_eef.urdf (robot description, URDF)
Before this commit: robot ur5, 10 links, 9 joints
Joints:
- joint ee_fixed_joint: origin xyz=0.0 0.0823 0.0 rpy=0.0 0.0 1.570796325 -> xyz=0.0 0.0823 0.0 rpy=-1.570796325 0.0 1.570796325
- joint sensor_ee_joint: origin xyz=0.14751 0.0 0.0 rpy=0.0 -1.57 0.0 -> xyz=0.184751 0.0 0.0 rpy=0.0 -1.57 0.0
