Commit message: Added force torque sensor model

File: sensor_description/urdf/ur5_force_eef.urdf (robot description, URDF)
Before this commit: robot ur5, 11 links, 10 joints
Joints:
- joint force_sensor_ee_joint: origin xyz=0.184751 0.0 0.0 rpy=0.0 -1.57 0.0 -> xyz=0.0495 0.0 0.0 rpy=0.0 1.5708 0.0
- joint sensor_ee_joint: origin xyz=0.184751 0.0 0.0 rpy=0.0 -1.57 0.0 -> xyz=0.0 0.0 0.184751 rpy=3.1415926 0.0 0.0

Commit message: Trying to import connector between the ft sensor and the US probe

File: sensor_description/urdf/ur5_force_eef.urdf (robot description, URDF)
Before this commit: robot ur5, 11 links, 10 joints
Links:
- added link connector, mass 0.05597; collision mesh filename=package://connector/meshes/connector.STL; visual mesh filename=package://connector/meshes/connector.STL

Commit message: Added connector between force sensor and US probe & Passed the test of active_echo_localization.cpp with ur5_force_old.launch

File: sensor_description/urdf/ur5_force_eef.urdf (robot description, URDF)
Before this commit: robot ur5, 12 links, 10 joints
Links:
- link connector: geometry collision mesh filename=package://connector_description/meshes/connector.STL; visual mesh filename=package://connector_description/meshes/connector.STL
Joints:
- added joint connector_force_sensor_joint: type fixed, parent robotiq_sensor_ft_150, child connector, origin xyz=0.0 0.0 0.0 rpy=0.0  0.0 0.0
- joint sensor_ee_joint: origin xyz=0.0 0.0 0.184751 rpy=3.1415926 0.0 0.0 -> xyz=0.0 0.0 0.200620 rpy=3.1415926 0.0 0.0; parent robotiq_sensor_ft_150 -> connector

Commit message: Readjust the sensors' orientations to beconsistent with real experiment setting

File: sensor_description/urdf/ur5_force_eef.urdf (robot description, URDF)
Before this commit: robot ur5, 12 links, 11 joints
Joints:
- joint force_sensor_ee_joint: origin xyz=0.0495 0.0 0.0 rpy=0.0 1.5708 0.0 -> xyz=0.0495 0.0 0.0 rpy=3.1415926 -1.570796325 0.0
- joint sensor_ee_joint: origin xyz=0.0 0.0 0.200620 rpy=3.1415926 0.0 0.0 -> xyz=0.0 0.0 0.200620 rpy=3.1415926 0.0 1.570796325

Commit message: Readjusted the orientations of the sensor to be consistent with real setup & Problem with testing simple_ur_driver and tra_simple_motion.cpp with active_echo_simul_keyboard

File: sensor_description/urdf/ur5_force_eef.urdf (robot description, URDF)
Before this commit: robot ur5, 12 links, 11 joints
Joints:
- joint force_sensor_ee_joint: origin xyz=0.0495 0.0 0.0 rpy=3.1415926 -1.570796325 0.0 -> xyz=0.0495 0.0 0.0 rpy=-1.570796325 0.0 -1.570796325
