Commit message: Successfully display robotiq force torque sensor

File: robotiq_sensor_ft_150/robots/robotiq_sensor_ft_150.urdf (robot description, URDF)
Before this commit: robot Robotiq_Sensor_FT_150, 1 links, 0 joints
Links:
- link base_link: geometry collision mesh filename=package://robotiq_sensor_ft_150/meshes/base_link.STL; visual mesh filename=package://robotiq_sensor_ft_150/meshes/base_link.STL
